File: power.kicad_sch (KiCad schematic)
At the start: 28 parts, among them J1 USB_C_Receptacle_PowerOnly_6P, J2 Conn_01x02_Pin, U3 TPD1E10B06DPYR, U4 BQ24073RGTR, U5 TPS63020DSJR, U6 TPD1E10B06DPYR

Commit message: PCB WIP
Parts:
- J2: value Conn_01x02_Pin -> PH 2.0 Horizontal
Other:
- moved on the sheet: J2, TP1, U6
Changed lines of the file:
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@@
 	)
 	(junction
-		(at 118.11 116.84)
+		(at 124.46 120.65)
 		(diameter 0)
 		(color 0 0 0 0)
@@
 	)
 	(junction
-		(at 121.92 116.84)
+		(at 128.27 120.65)
 		(diameter 0)
 		(color 0 0 0 0)
@@
 	)
 	(junction
-		(at 119.38 121.92)
+		(at 125.73 125.73)
 		(diameter 0)
 		(color 0 0 0 0)
@@
 	(wire
 		(pts
-			(xy 119.38 121.92) (xy 121.92 121.92)
+			(xy 125.73 125.73) (xy 128.27 125.73)
 		)
 		(stroke
@@
 	(wire
 		(pts
-			(xy 119.38 127) (xy 119.38 121.92)
+			(xy 125.73 130.81) (xy 125.73 125.73)
 		)
 		(stroke
@@
 	(wire
 		(pts
-			(xy 121.92 116.84) (xy 130.81 116.84)
+			(xy 128.27 120.65) (xy 137.16 120.65)
 		)
 		(stroke
@@
 	(wire
 		(pts
-			(xy 119.38 119.38) (xy 119.38 121.92)
+			(xy 125.73 123.19) (xy 125.73 125.73)
 		)
 		(stroke
@@
 	(wire
 		(pts
-			(xy 118.11 116.84) (xy 113.03 116.84)
+			(xy 124.46 120.65) (xy 119.38 120.65)
 		)
 		(stroke
@@
 	(wire
 		(pts
-			(xy 121.92 116.84) (xy 118.11 116.84)
+			(xy 128.27 120.65) (xy 124.46 120.65)
 		)
 		(stroke
@@
 	(wire
 		(pts
-			(xy 113.03 119.38) (xy 119.38 119.38)
+			(xy 119.38 123.19) (xy 125.73 123.19)
 		)
 		(stroke
@@
 	)
 	(label "VBAT"
-		(at 130.81 116.84 180)
+		(at 137.16 120.65 180)
 		(fields_autoplaced yes)
 		(effects
@@
 		)
 		(property "Net Class" "power"
-			(at 130.81 118.11 0)
+			(at 137.16 121.92 0)
 			(hide yes)
 			(show_name no)
@@
 	(symbol
 		(lib_id "Muffin_DIODES:TPD1E10B06DPYR")
-		(at 121.92 105.41 270)
+		(at 128.27 109.22 270)
 		(unit 1)
 		(body_style 1)
@@
 		(fields_autoplaced yes)
 		(property "Reference" "U6"
-			(at 124.46 118.7449 90)
+			(at 130.81 122.5549 90)
 			(show_name no)
 			(do_not_autoplace no)
@@
 		)
 		(property "Value" "TPD1E10B06DPYR"
-			(at 124.46 120.65 90)
+			(at 130.81 124.46 90)
 			(show_name no)
 			(do_not_autoplace no)
@@
 		)
 		(property "Footprint" "Muffin_SMD:X1SON-2_L1.0-W0.6-P0.65-BI"
-			(at 116.586 119.38 0)
+			(at 122.936 123.19 0)
 			(hide yes)
 			(show_name no)
@@
 		)
 		(property "Datasheet" "TPD1E10B06DPYR"
-			(at 118.618 119.38 0)
+			(at 124.968 123.19 0)
 			(hide yes)
 			(show_name no)
@@
 		)
 		(property "Description" ""
-			(at 121.92 105.41 0)
+			(at 128.27 109.22 0)
 			(hide yes)
 			(show_name no)
@@
 		)
 		(property "LCSC" "C48260"
-			(at 114.554 119.38 0)
+			(at 120.904 123.19 0)
 			(hide yes)
 			(show_name no)
@@
 	(symbol
 		(lib_id "Connector:TestPoint")
-		(at 118.11 116.84 0)
+		(at 124.46 120.65 0)
 		(unit 1)
 		(body_style 1)
@@
 		(fields_autoplaced yes)
 		(property "Reference" "TP1"
-			(at 120.65 112.2679 0)
+			(at 127 116.0779 0)
 			(show_name no)
 			(do_not_autoplace no)
@@
 		)
 		(property "Value" "VBAT"
-			(at 120.65 114.8079 0)
+			(at 127 118.6179 0)
 			(show_name no)
 			(do_not_autoplace no)
@@
 		)
 		(property "Footprint" "TestPoint:TestPoint_Pad_D1.0mm"
-			(at 123.19 116.84 0)
+			(at 129.54 120.65 0)
 			(hide yes)
 			(show_name no)
@@
 		)
 		(property "Datasheet" ""
-			(at 123.19 116.84 0)
+			(at 129.54 120.65 0)
 			(hide yes)
 			(show_name no)
@@
 		)
 		(property "Description" "test point"
-			(at 118.11 116.84 0)
+			(at 124.46 120.65 0)
 			(hide yes)
 			(show_name no)
@@
 	(symbol
 		(lib_id "Connector:Conn_01x02_Pin")
-		(at 107.95 119.38 0)
+		(at 114.3 123.19 0)
 		(mirror x)
 		(unit 1)
@@
 		(in_pos_files yes)
 		(dnp no)
+		(fields_autoplaced yes)
 		(property "Reference" "J2"
-			(at 108.585 124.46 0)
+			(at 113.03 120.6499 0)
 			(show_name no)
 			(do_not_autoplace no)
@@
 					(size 1.27 1.27)
 				)
+				(justify right)
 			)
 		)
-		(property "Value" "Conn_01x02_Pin"
-			(at 108.585 121.92 0)
+		(property "Value" "PH 2.0 Horizontal"
+			(at 113.03 123.1899 0)
 			(show_name no)
 			(do_not_autoplace no)
@@
 					(size 1.27 1.27)
 				)
+				(justify right)
 			)
 		)
 		(property "Footprint" "Connector_Muffin_THT:JST_PH_S2B-PH-K_1x02_P2.00mm_Horizontal"
-			(at 107.95 119.38 0)
+			(at 114.3 123.19 0)
 			(hide yes)
 			(show_name no)
@@
 		)
 		(property "Datasheet" ""
-			(at 107.95 119.38 0)
+			(at 114.3 123.19 0)
 			(hide yes)
 			(show_name no)
@@
 		)
 		(property "Description" "Generic connector, single row, 01x02, script generated"
-			(at 107.95 119.38 0)
+			(at 114.3 123.19 0)
 			(hide yes)
 			(show_name no)
@@
 	(symbol
 		(lib_id "power:GND")
-		(at 119.38 127 0)
+		(at 125.73 130.81 0)
 		(mirror y)
 		(unit 1)
@@
 		(fields_autoplaced yes)
 		(property "Reference" "#PWR021"
-			(at 119.38 133.35 0)
+			(at 125.73 137.16 0)
 			(hide yes)
 			(show_name no)
@@
 		)
 		(property "Value" "GND"
-			(at 119.38 132.08 0)
+			(at 125.73 135.89 0)
 			(show_name no)
 			(do_not_autoplace no)
@@
 		)
 		(property "Footprint" ""
-			(at 119.38 127 0)
+			(at 125.73 130.81 0)
 			(hide yes)
 			(show_name no)
@@
 		)
 		(property "Datasheet" ""
-			(at 119.38 127 0)
+			(at 125.73 130.81 0)
 			(hide yes)
 			(show_name no)
@@
 		)
 		(property "Description" "Power symbol creates a global label with name \"GND\" , ground"
-			(at 119.38 127 0)
+			(at 125.73 130.81 0)
 			(hide yes)
 			(show_name no)
