File: uAir.kicad_sch (KiCad schematic)
At the start: 35 parts, among them Q1 DTC143Z, Q2 DTC143Z, Q3 DTC143Z, Q4 DTC143Z, SW1 SW_Push, U1 BME680, U2 STM32G031G8Ux

Commit message: PCB WIP
Parts:
- removed C11, C12, C14: 0.1u, Capacitor_SMD:C_0402_1005Metric, symbol Device:C
- removed RN1: 300, Resistor_SMD:R_Array_Convex_4x0402, symbol Device:R_Pack04
- added D5: SS34, Diode_SMD:D_SMA, symbol Diode:SS34
- added J3, J4: PicoBlade 1x4p, Connector_Molex:Molex_PicoBlade_53261-0471_1x04-1MP_P1.25mm_Horizontal, symbol Connector_Generic_MountingPin:Conn_01x04_MountingPin
- added J5: PLS 2.54 1x4p Vertical, Connector_PinHeader_2.54mm:PinHeader_1x04_P2.54mm_Vertical, symbol Connector:Conn_01x04_Pin
- added J6: PicoBlade 1x5p, Connector_Molex:Molex_PicoBlade_53261-0571_1x05-1MP_P1.25mm_Horizontal, symbol Connector_Generic_MountingPin:Conn_01x05_MountingPin
- added J7: PicoBlade 1x8p, Connector_Molex:Molex_PicoBlade_53261-0871_1x08-1MP_P1.25mm_Horizontal, symbol Connector_Generic_MountingPin:Conn_01x08_MountingPin
- added R16, R17, R18, R19, R20: 300, Resistor_SMD:R_0603_1608Metric, symbol Device:R
- added R21: 10k, Resistor_SMD:R_0603_1608Metric, symbol Device:R
- added TP12: SPI2_SCK, TestPoint:TestPoint_THTPad_D1.0mm_Drill0.5mm, symbol Connector:TestPoint
- added TP13, TP22: PA1, TestPoint:TestPoint_THTPad_D1.0mm_Drill0.5mm, symbol Connector:TestPoint
- added TP14: TX, TestPoint:TestPoint_THTPad_D1.0mm_Drill0.5mm, symbol Connector:TestPoint
- added TP15: RX, TestPoint:TestPoint_THTPad_D1.0mm_Drill0.5mm, symbol Connector:TestPoint
- added TP16, TP21: SPI2_MOSI, TestPoint:TestPoint_THTPad_D1.0mm_Drill0.5mm, symbol Connector:TestPoint
- added TP17: SWDIO, TestPoint:TestPoint_THTPad_D1.0mm_Drill0.5mm, symbol Connector:TestPoint
- added TP18: SWCLK, TestPoint:TestPoint_THTPad_D1.0mm_Drill0.5mm, symbol Connector:TestPoint
- added TP19, TP20: GND, TestPoint:TestPoint_THTPad_D1.0mm_Drill0.5mm, symbol Connector:TestPoint
- added TP23: LED_R, TestPoint:TestPoint_THTPad_D1.0mm_Drill0.5mm, symbol Connector:TestPoint
- added TP24: LED_G, TestPoint:TestPoint_THTPad_D1.0mm_Drill0.5mm, symbol Connector:TestPoint
- added TP25: LED_B, TestPoint:TestPoint_THTPad_D1.0mm_Drill0.5mm, symbol Connector:TestPoint
- added U7: TPD4E05U06DQA, Package_SON:USON-10_2.5x1.0mm_P0.5mm, symbol Power_Protection:TPD4E05U06DQA
- C15: value 0.1u -> 1u; footprint Capacitor_SMD:C_0402_1005Metric -> Capacitor_SMD:C_0603_1608Metric
- D4: LCSC (none) -> C125110
- Q2, Q3, Q4: footprint Muffin_SMD:SOT-523 -> Package_TO_SOT_SMD:SC-59
- SW1: footprint Button_Switch_SMD:SW_Push_1P1T_NO_E-Switch_TL3301NxxxxxG -> Muffin_THT:SW_Kailh_Choc_V1V2_Led
- TP10: value SDA -> SDA1
- TP4: value SCL -> SCL2
- TP5: value SDA -> SDA2
- TP9: value SCL -> SCL1
- U2: footprint Muffin_SMD:QFN-28_4x4mm_P0.5mm -> Package_DFN_QFN:QFN-28_4x4mm_P0.5mm
Connections:
- net +3V3: now also D5.1 (K), J3.1 (Pin_1), J4.1 (Pin_1), J5.1 (Pin_1), J7.8 (Pin_8); no longer D2.5 (VCC)
- net BTN: now also U2.2 (PC15)
- net GND: now also J3.4 (Pin_4), J3.MP (MountPin), J4.4 (Pin_4), J4.MP (MountPin), J5.4 (Pin_4), J6.3 (Pin_3), J6.MP (MountPin), J7.7 (Pin_7), J7.MP (MountPin), TP19.1, TP20.1, U7.3 (GND), U7.8 (GND)
- net LED_B: now also U2.25 (PB5), TP25.1
- net LED_G: now also U2.24 (PB4), TP24.1
- net LED_R: now also U2.15 (PB1), TP23.1
- net RESET: now also J6.1 (Pin_1)
- net RX: now also U2.22 (PA15), R20.2, TP21.1, U7.5 (D2-), U7.6 (NC); no longer TP10.1, U2.27 (PB7)
- net SWCLK: now also J6.4 (Pin_4), TP18.1
- net SWDIO: now also J6.2 (Pin_2), TP17.1
- net TX: now also U2.8 (PA2), R19.2, TP14.1, U7.4 (D2+), U7.7 (NC); no longer TP9.1, U2.26 (PB6)
- net VSYS: now also R21.2
- net en: now also R21.1
- net latch: now also U2.1 (PC14)
- net at D4.3 (BK): now also R18.1
- net at D4.2 (GK): now also R17.1
- net at D4.1 (RK): now also R16.1
- net at Q4.3 (C): now also R16.2
- net at Q3.3 (C): now also R17.2
- net at Q2.3 (C): now also R18.2
- net D/C: now reaches U2.10 (PA4)
- net D/C: now also J7.3 (Pin_3), TP16.1
- net SPI2_CS: now reaches U2.16 (PA8)
- net SPI2_CS: now also J7.4 (Pin_4), TP22.1
- net BL/RES: now reaches U2.17 (PC6)
- net BL/RES: now also J7.1 (Pin_1)
- net PGOOD: now reaches U2.23 (PB3)
- net CHRG: now reaches U2.28 (PB8)
- net SPI2_SCK: now reaches U2.6 (PA0)
- net SPI2_SCK: now also J7.5 (Pin_5), TP12.1
- net DISP_RST: now reaches U2.7 (PA1)
- net DISP_RST: now also J7.2 (Pin_2), TP13.1
- net SPI2_MOSI: now reaches U2.9 (PA3)
- net SPI2_MOSI: now also J7.6 (Pin_6), TP15.1
- net SCL renamed SCL2
- net SCL2: now also J3.2 (Pin_2), U7.1 (D1+), U7.10 (NC)
- net SDA renamed SDA2
- net SDA2: now also J3.3 (Pin_3), U7.2 (D1-), U7.9 (NC)
- new net: J4.3 (Pin_3), R20.1
- new net: J4.2 (Pin_2), R19.1
- new net DBG_VCC: D2.5 (VCC), D5.2 (A), J6.5 (Pin_5)
- new net SCL1: J5.2 (Pin_2), TP9.1, U2.26 (PB6)
- new net SDA1: J5.3 (Pin_3), TP10.1, U2.27 (PB7)
- no-connect marks 2 -> 0
Other:
- moved on the sheet: C1, C13, C15, C16, D1, D2, D3, DISP1, Q1, Q2, Q3, Q4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

Commit message: Sync
Parts:
- removed TP10: SDA1, TestPoint:TestPoint_THTPad_D1.0mm_Drill0.5mm, symbol Connector:TestPoint
- removed TP12: SPI2_SCK, TestPoint:TestPoint_THTPad_D1.0mm_Drill0.5mm, symbol Connector:TestPoint
- removed TP13, TP22: PA1, TestPoint:TestPoint_THTPad_D1.0mm_Drill0.5mm, symbol Connector:TestPoint
- removed TP15: RX, TestPoint:TestPoint_THTPad_D1.0mm_Drill0.5mm, symbol Connector:TestPoint
- removed TP16: SPI2_MOSI, TestPoint:TestPoint_THTPad_D1.0mm_Drill0.5mm, symbol Connector:TestPoint
- removed TP4: SCL2, TestPoint:TestPoint_THTPad_D1.0mm_Drill0.5mm, symbol Connector:TestPoint
- removed TP5: SDA2, TestPoint:TestPoint_THTPad_D1.0mm_Drill0.5mm, symbol Connector:TestPoint
- removed TP9: SCL1, TestPoint:TestPoint_THTPad_D1.0mm_Drill0.5mm, symbol Connector:TestPoint
- TP21: value SPI2_MOSI -> RX
