File: uAir.kicad_pcb (KiCad board)
At the start: 2 copper layers, 58 parts, among them J1 USB_C_Receptacle_PowerOnly_6P, J2 Conn_01x02_Pin, Q1 DTC143Z, SW1 SW_Push, SW2 SW_SPDT_SH, U1 BME680, U2 STM32G031G8Ux, U3 TPD1E10B06DPYR, U4 BQ24073RGTR, U5 TPS63020DSJR, U6 TPD1E10B06DPYR

Commit message: PCB WIP
Parts:
- removed C11, C12, C14: 0.1u, Capacitor_SMD:C_0402_1005Metric
- removed SW2: SW_SPDT_SH, Muffin_SMD:MSK12C02
- added D3: 1N4148WS, Diode_SMD:D_SOD-323, F.Cu at (164.2, 82.0)
- added D4: LED_RGBA, LED_SMD:LED_LiteOn_LTST-C19HE1WT, F.Cu at (148.4, 86.2)
- added D5: SS34, Diode_SMD:D_SMA, F.Cu at (148.8, 99.2)
- added J3: PicoBlade 1x4p, Connector_Molex:Molex_PicoBlade_53261-0471_1x04-1MP_P1.25mm_Horizontal, F.Cu at (141.0, 73.0)
- added J4: PicoBlade 1x4p, Connector_Molex:Molex_PicoBlade_53261-0471_1x04-1MP_P1.25mm_Horizontal, F.Cu at (141.0, 85.0)
- added J5: PLS 2.54 1x4p Vertical, Connector_PinHeader_2.54mm:PinHeader_1x04_P2.54mm_Vertical, F.Cu at (161.0, 106.2)
- added J6: PicoBlade 1x5p, Connector_Molex:Molex_PicoBlade_53261-0571_1x05-1MP_P1.25mm_Horizontal, F.Cu at (141.0, 97.6)
- added J7: PicoBlade 1x8p, Connector_Molex:Molex_PicoBlade_53261-0871_1x08-1MP_P1.25mm_Horizontal, F.Cu at (153.4, 41.8)
- added Q2: DTC143Z, Package_TO_SOT_SMD:SC-59, F.Cu at (172.0, 71.4)
- added Q3: DTC143Z, Package_TO_SOT_SMD:SC-59, F.Cu at (172.0, 75.0)
- added Q4: DTC143Z, Package_TO_SOT_SMD:SC-59, F.Cu at (172.0, 67.8)
- added R16: 300, Resistor_SMD:R_0603_1608Metric, F.Cu at (175.4, 67.8)
- added R17: 300, Resistor_SMD:R_0603_1608Metric, F.Cu at (175.4, 75.0)
- added R18: 300, Resistor_SMD:R_0603_1608Metric, F.Cu at (175.4, 71.4)
- added R19: 300, Resistor_SMD:R_0603_1608Metric, F.Cu at (145.6, 77.4)
- added R20: 300, Resistor_SMD:R_0603_1608Metric, F.Cu at (147.2, 77.4)
- added R21: 10k, Resistor_SMD:R_0603_1608Metric, F.Cu at (169.0, 93.8)
- added TP12: SPI2_SCK, TestPoint:TestPoint_THTPad_D1.0mm_Drill0.5mm, F.Cu at (203.8, 44.0)
- added TP13: PA1, TestPoint:TestPoint_THTPad_D1.0mm_Drill0.5mm, F.Cu at (210.2, 44.0)
- added TP14: TX, TestPoint:TestPoint_THTPad_D1.0mm_Drill0.5mm, F.Cu at (183.0, 60.6)
- added TP15: RX, TestPoint:TestPoint_THTPad_D1.0mm_Drill0.5mm, F.Cu at (191.0, 60.8)
- added TP16: SPI2_MOSI, TestPoint:TestPoint_THTPad_D1.0mm_Drill0.5mm, F.Cu at (207.0, 44.0)
- added TP17: SWDIO, TestPoint:TestPoint_THTPad_D1.0mm_Drill0.5mm, F.Cu at (198.6, 53.6)
- added TP18: SWCLK, TestPoint:TestPoint_THTPad_D1.0mm_Drill0.5mm, F.Cu at (133.0, 83.8)
- added TP19: GND, TestPoint:TestPoint_THTPad_D1.0mm_Drill0.5mm, B.Cu at (118.9, 32.8)
- added TP20: GND, TestPoint:TestPoint_THTPad_D1.0mm_Drill0.5mm, B.Cu at (129.1, 30.2)
- added TP21: SPI2_MOSI, TestPoint:TestPoint_THTPad_D1.0mm_Drill0.5mm, F.Cu at (115.7, 64.6)
- added TP22: PA1, TestPoint:TestPoint_THTPad_D1.0mm_Drill0.5mm, F.Cu at (112.6, 64.6)
- added TP23: LED_R, TestPoint:TestPoint_THTPad_D1.0mm_Drill0.5mm, F.Cu at (109.5, 64.6)
- added TP24: LED_G, TestPoint:TestPoint_THTPad_D1.0mm_Drill0.5mm, F.Cu at (106.5, 64.6)
- added TP25: LED_B, TestPoint:TestPoint_THTPad_D1.0mm_Drill0.5mm, F.Cu at (103.5, 64.6)
- added U7: TPD4E05U06DQA, Package_SON:USON-10_2.5x1.0mm_P0.5mm, F.Cu at (147.6, 74.4)
- C15: value 0.1u -> 1u; footprint Capacitor_SMD:C_0402_1005Metric -> Capacitor_SMD:C_0603_1608Metric
- D2, DISP1: moved to B.Cu
- J2: value Conn_01x02_Pin -> PH 2.0 Horizontal
- SW1: footprint Button_Switch_SMD:SW_Push_1P1T_NO_E-Switch_TL3301NxxxxxG -> Muffin_THT:SW_Kailh_Choc_V1V2_Led; moved to B.Cu
- TP10: value SDA -> SDA1
- TP11: footprint TestPoint:TestPoint_THTPad_D1.0mm_Drill0.5mm -> TestPoint:TestPoint_Pad_D1.0mm
- TP4: value SCL -> SCL2
- TP5: value SDA -> SDA2
- TP9: value SCL -> SCL1
- U2: footprint Muffin_SMD:QFN-28_4x4mm_P0.5mm -> Package_DFN_QFN:QFN-28_4x4mm_P0.5mm
- moved TP6 81.2 mm to (110.8, 34.9), turned to 180 degrees
- moved R10 70.2 mm to (179.8, 95.6)
- moved TP1 69.6 mm to (107.6, 38.4), turned to 180 degrees
- moved R9 69.6 mm to (179.8, 97.2)
- moved TP2 69.3 mm to (110.8, 41.0), turned to 180 degrees
- moved C2 68.3 mm to (179.0, 92.8), turned to 90 degrees
- moved J2 66.9 mm to (186.6, 98.0), turned to 180 degrees
- moved C3 65.1 mm to (175.8, 96.8)
- moved R12 63.2 mm to (173.0, 102.2), turned to -90 degrees
- moved C4 62.8 mm to (173.0, 92.8), turned to 90 degrees
- moved R8 62.7 mm to (173.0, 96.0), turned to -90 degrees
- moved R11 62.5 mm to (173.0, 105.2), turned to 90 degrees
- moved J1 60.8 mm to (179.2, 104.6)
- moved U1 56.3 mm to (178.2, 51.6)
- moved C6 55.8 mm to (169.5, 96.3), turned to -90 degrees
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Connections:
- net /SCL renamed /SCL2
- net /SDA renamed /SDA2
- D1 pad 2: /latch -> /SWITCH
- D2 pad 5: +3V3 -> /DBG_VCC
- TP10 pad 1: /RX -> /SDA1
- TP9 pad 1: /TX -> /SCL1
- U2 pad 1: unconnected-(U2-PC14-Pad1) -> /latch
- U2 pad 10: unconnected-(U2-PA4-Pad10) -> /D/C
- U2 pad 15: unconnected-(U2-PB1-Pad15) -> /LED_R
- U2 pad 16: unconnected-(U2-PA8-Pad16) -> /SPI2_CS
- U2 pad 17: unconnected-(U2-PC6-Pad17) -> /BL/RES
- U2 pad 2: unconnected-(U2-PC15-Pad2) -> /BTN
- U2 pad 22: unconnected-(U2-PA15-Pad22) -> /RX
- U2 pad 23: unconnected-(U2-PB3-Pad23) -> /PGOOD
- U2 pad 24: unconnected-(U2-PB4-Pad24) -> /LED_G
- U2 pad 25: unconnected-(U2-PB5-Pad25) -> /LED_B
- U2 pad 26: /TX -> /SCL1
- U2 pad 27: /RX -> /SDA1
- U2 pad 28: unconnected-(U2-PB8-Pad28) -> /CHRG
- U2 pad 6: unconnected-(U2-PA0-Pad6) -> /SPI2_SCK
- U2 pad 7: unconnected-(U2-PA1-Pad7) -> /DISP_RST
- U2 pad 8: unconnected-(U2-PA2-Pad8) -> /TX
- U2 pad 9: unconnected-(U2-PA3-Pad9) -> /SPI2_MOSI
- U4 pad 7: /power/PGOOD -> /PGOOD
- U4 pad 9: /power/CHRG -> /CHRG
Routing:
- net /SPI2_SCK: track 0.00 -> 80.9 mm
- net /SPI2_MOSI: track 0.00 -> 80.0 mm
- net /RESET: track 0.00 -> 72.8 mm, vias 0 -> 3
- net /SWDIO: track 0.00 -> 56.4 mm, vias 0 -> 3
- net /SWCLK: track 0.00 -> 50.1 mm, vias 0 -> 3
- net /SPI_CS: track 0.00 -> 46.4 mm, vias 0 -> 3
- net /BL/RES: track 0.00 -> 42.8 mm, vias 0 -> 2
- net /MOSI: track 0.00 -> 42.6 mm
- net /SPI_CLK: track 0.00 -> 42.1 mm
- net /TX: track 0.00 -> 40.2 mm, vias 0 -> 1
- net /RX: track 0.00 -> 39.6 mm, vias 0 -> 1
- net /MISO: track 0.00 -> 38.5 mm
- net /DISP_RST: track 0.00 -> 38.3 mm, vias 0 -> 2
- net Net-(D4-BK): track 0.00 -> 37.2 mm, vias 0 -> 2
- net /SCL2: track 0.00 -> 37.0 mm
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Other:
- board outline added: 51.2 x 69.4 mm
- copper layers 2 -> 4

Commit message: Sync
Parts:
- removed TP10: SDA1, TestPoint:TestPoint_THTPad_D1.0mm_Drill0.5mm
- removed TP12: SPI2_SCK, TestPoint:TestPoint_THTPad_D1.0mm_Drill0.5mm
- removed TP13, TP22: PA1, TestPoint:TestPoint_THTPad_D1.0mm_Drill0.5mm
- removed TP15: RX, TestPoint:TestPoint_THTPad_D1.0mm_Drill0.5mm
- removed TP16: SPI2_MOSI, TestPoint:TestPoint_THTPad_D1.0mm_Drill0.5mm
- removed TP4: SCL2, TestPoint:TestPoint_THTPad_D1.0mm_Drill0.5mm
- removed TP5: SDA2, TestPoint:TestPoint_THTPad_D1.0mm_Drill0.5mm
- removed TP9: SCL1, TestPoint:TestPoint_THTPad_D1.0mm_Drill0.5mm
- D4: moved to B.Cu
- TP21: value SPI2_MOSI -> RX
- moved TP11 87.0 mm to (171.0, 81.2)
- moved TP8 83.3 mm to (169.8, 88.6), turned to 0 degrees
- moved TP6 81.1 mm to (173.2, 86.6)
- moved TP1 79.9 mm to (173.2, 84.0)
- moved TP20 76.7 mm to (161.4, 99.8)
- moved TP2 75.5 mm to (171.0, 86.6)
- moved TP19 72.7 mm to (173.2, 81.2)
- moved TP17 52.8 mm to (150.4, 75.2)
- moved TP7 43.3 mm to (164.2, 69.2)
- moved TP14 41.0 mm to (145.6, 77.4), turned to 0 degrees
- moved TP21 34.6 mm to (147.8, 77.4), turned to 0 degrees
- moved TP18 21.2 mm to (152.4, 75.2), turned to 0 degrees
- moved TP3 20.4 mm to (171.0, 84.0)
- moved J2 12.2 mm to (179.6, 88.0)
- moved TP24 5.39 mm to (106.2, 70.0)
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Routing:
- net +3V3: track 30.1 -> 209.4 mm, vias 0 -> 25
- net /TX: track 40.2 -> 55.0 mm, vias 1 -> 2
- net /DBG_VCC: track 0.00 -> 14.0 mm, vias 0 -> 4
- net /SWDIO: track 56.4 -> 44.8 mm, vias 3 -> 2
- net /en: track 6.22 -> 16.6 mm
- net GND: track 9.15 -> 19.0 mm, vias 1 -> 32
- net /SPI2_SCK: track 80.9 -> 72.5 mm
- net VSYS: track 15.2 -> 6.71 mm, vias 2 -> 1
- net /SPI2_MOSI: track 80.0 -> 72.9 mm
- net /SWCLK: track 50.1 -> 43.4 mm, vias 3 -> 2
- net /DISP_RST: track 38.3 -> 32.5 mm
- net /SPI2_CS: track 36.3 -> 30.9 mm
- net Net-(D4-RK): track 36.5 -> 41.4 mm, vias 2 -> 1
- net /SPI_CS: track 46.4 -> 51.3 mm
- net /MISO: track 38.5 -> 33.9 mm
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- added copper zone on B.Cu, net +3V3
- added copper zone on F.Cu, net +3V3
- added copper zone on F.Cu, net /power/VBAT
- added copper zone on F.Cu, net /power/VBUS
- added copper zone on F.Cu, net GND
- added copper zone on In1.Cu, net GND
- added copper zone on In2.Cu, net GND
- added copper zone on F.Cu, net Net-(L1-Pad1)
- added copper zone on F.Cu, net Net-(L1-Pad2)
- added copper zone on F.Cu, net VSYS
Other:
- board size 51.2 x 69.4 mm -> 43.8 x 70.2 mm

Commit message: Finished PCB
Parts:
- TP19, TP20: moved to F.Cu
- moved TP25 68.3 mm to (168.6, 71.5)
- moved TP23 62.7 mm to (168.6, 67.8)
- moved TP24 62.6 mm to (168.6, 75.0)
- moved U6 2.60 mm to (180.0, 90.6), turned to 0 degrees
- moved R21 1.88 mm to (169.2, 90.8), turned to -90 degrees
- moved TP8 1.34 mm to (171.0, 89.2)
- moved C2 0.82 mm to (179.8, 93.0), turned to 0 degrees
- moved TH1 0.63 mm to (180.2, 94.4)
- moved R11 0.20 mm to (170.2, 105.2)
- moved R12 0.20 mm to (170.2, 102.2)
- moved R10 0.20 mm to (179.8, 95.8)
- moved R9 0.20 mm to (179.8, 97.4)
- moved J1 0.20 mm to (176.4, 104.6)
- turned TP19 to 180 degrees
- turned TP20 to 180 degrees
Routing:
- net GND: track 19.0 -> 67.1 mm, vias 32 -> 123
- net +3V3: track 209.4 -> 243.5 mm
- net VSYS: track 6.71 -> 31.4 mm, vias 1 -> 9
- net /power/VBUS: track 0.00 -> 15.8 mm, vias 0 -> 2
- net /power/VBAT: track 0.00 -> 8.00 mm, vias 0 -> 1
- net /BTN: track 18.0 -> 22.5 mm
- net /SWITCH: track 14.2 -> 16.5 mm
- net /en: track 16.6 -> 18.7 mm
- net /SPI_CS: track 51.3 -> 49.3 mm
- net /D/C: track 33.2 -> 31.2 mm
- net /SPI_CLK: track 37.7 -> 35.9 mm
- net /BL/RES: track 40.8 -> 39.6 mm
- net /LED_R: track 23.2 -> 22.1 mm, vias 2 -> 1
- net /RESET: track 70.4 -> 71.3 mm
- net Net-(D4-RK): track 41.4 -> 42.3 mm
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- added copper zone on B.Cu, net VSYS
